File: Roboboat-PD2.kicad_sch (KiCad schematic)
At the start: 29 parts, among them J1 12V, J10 Motor, J11 Motor, J12 Motor, J13 Motor, J14 5V, J15 14.4V, J16 PGOOD, J2 Bucky, J3 Jetson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

Commit message: final touches
Parts:
- L1: value 440nH -> 150uH; footprint footprints:IND_PA0513_PUL -> footprints:IND_SRP1265A-1R5M
- SW1: renamed from SW2; footprint Connector_PinHeader_1.00mm:PinHeader_1x02_P1.00mm_Vertical -> Connector_PinHeader_2.54mm:PinHeader_1x02_P2.54mm_Vertical
Changed lines of the file:
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@@
 		(dnp no)
 		(fields_autoplaced yes)
-		(property "Reference" "SW2"
+		(property "Reference" "SW1"
 			(at 104.14 41.9099 90)
 			(effects
@@
 			)
 		)
-		(property "Footprint" "Connector_PinHeader_1.00mm:PinHeader_1x02_P1.00mm_Vertical"
+		(property "Footprint" "Connector_PinHeader_2.54mm:PinHeader_1x02_P2.54mm_Vertical"
 			(at 102.87 43.18 0)
 			(effects
@@
 			(project "Roboboat-PD2"
 				(path "/9a1496f4-7cef-4d33-8239-9c2f43ceb177"
-					(reference "SW2")
+					(reference "SW1")
 					(unit 1)
 				)
@@
 			)
 		)
-		(property "Value" "440nH"
+		(property "Value" "150uH"
 			(at 170.18 62.23 90)
 			(effects
@@
 			)
 		)
-		(property "Footprint" "footprints:IND_PA0513_PUL"
+		(property "Footprint" "footprints:IND_SRP1265A-1R5M"
 			(at 170.18 64.77 0)
 			(effects
